Commit message: Hexcopter URDF

File: gym_pybullet_drones/assets/hexcopter.urdf (robot description, URDF)
Before this commit: robot cf2, 6 links, 5 joints
Links:
- link base_link: geometry collision cylinder length=.025 radius=.06; visual mesh filename=./hexcopter.stl scale=0.001 0.001 0.001

Commit message: hexcopter collision stl

File: gym_pybullet_drones/assets/hexcopter.urdf (robot description, URDF)
Before this commit: robot cf2, 6 links, 5 joints
Links:
- link base_link: geometry collision mesh filename=./hexcopter.stl scale=0.001 0.001 0.001; visual mesh filename=./hexcopter_s.stl scale=0.001 0.001 0.001

Commit message: Hexacopter dynamics

File: gym_pybullet_drones/assets/hexcopter.urdf (robot description, URDF)
Before this commit: robot cf2, 6 links, 5 joints
Links:
- added link prop4_link, mass 0
- added link prop5_link, mass 0
- link base_link: mass 0.027 -> 0.65; geometry collision mesh filename=./hexcopter_stl.stl scale=1 1 1; visual mesh filename=./hexcopter_stl.stl scale=1 1 1
Joints:
- added joint prop4_joint: type fixed, parent base_link, child prop4_link
- added joint prop5_joint: type fixed, parent base_link, child prop5_link
